File: Test Board/Test Board/new_clamp_anti_windup.kicad_sch (KiCad schematic)
At the start: 31 parts, among them U10 BUF634A, U11 OPA189, U12 OPA189, U13 OPA189, U7 OPA189, U8 OPA189, U9 OPA189

Commit message: First pass at routing Test Board, TODO: Find and Double check Part numbers
Parts:
- added C19, C20, C21, C22, C23, C24, C26, C27, C28, C29, C30, C31, C34, C35: 100nF, Capacitor_SMD:C_0805_2012Metric, symbol Device:C
- renumbered C30 to C18, C31 to C25, C34 to C36
Connections:
- net +15V: now also C19.1, C21.1, C23.1, C27.1, C28.2, C30.1, C34.1
- net -15V: now also C20.1, C22.1, C24.1, C26.2, C29.1, C31.1, C35.1
- net GND: now also C19.2, C20.2, C21.2, C22.2, C23.2, C24.2, C26.1, C27.2, C28.1, C29.2, C30.2, C31.2, C34.2, C35.2
